File: ekg-interface/ekg-interface.kicad_sch (KiCad schematic)
At the start: 19 parts, among them J1 TRS Jack, J2 Screw_Terminal_01x02, J3 Screw_Terminal_01x02, U1 INA126P, U2 TL071

Commit message: images
Other:
- title: (none) -> EKG Interface
Changed lines of the file:
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@@
 	(generator_version "8.0")
 	(paper "A4")
+	(title_block
+		(title "EKG Interface")
+		(date "2025-02-01")
+		(rev "1.0")
+	)
 	(junction
 		(at 219.71 87.63)
