File: step-down/step-down.kicad_sch (KiCad schematic)
At the start: 20 parts, among them J0 1725656, J1 1725656, M1 IRF7413ZPBF, M2 IRF7413ZPBF, U1 LTC3807EFE-TRPBF

Commit message: images
Other:
- title: Buck Converter for EKG Project -> Step-down converter
Changed lines of the file:
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@@
 	(paper "A4")
 	(title_block
-		(title "Buck Converter for EKG Project")
+		(title "Step-down converter")
 	)
 	(junction

Commit message: set components
Parts:
- added C8: 47u, Capacitor_SMD:C_1210_3225Metric, symbol Device:C
- C7: value 150u -> 100u; footprint (none) -> Capacitor_SMD:C_1210_3225Metric
Connections:
- net GND: now also C8.2
- net at C7.1, J1.2 (Pin_2), R4.2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: now also C8.1
Other:
- moved on the sheet: J1
Changed lines of the file:
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@@
 	)
 	(junction
+		(at 236.22 128.27)
+		(diameter 0)
+		(color 0 0 0 0)
+	)
+	(junction
 		(at 208.28 128.27)
 		(diameter 0)
@@
 	(wire
 		(pts
-			(xy 229.87 68.58) (xy 229.87 74.93)
+			(xy 236.22 128.27) (xy 246.38 128.27)
 		)
 		(stroke
@@
 	(wire
 		(pts
-			(xy 224.79 128.27) (xy 224.79 77.47)
-		)
-		(stroke
-			(width 0)
-			(type default)
-		)
-	)
-	(wire
-		(pts
 			(xy 147.32 125.73) (xy 148.59 125.73)
 		)
@@
 	(wire
 		(pts
-			(xy 224.79 77.47) (xy 229.87 77.47)
-		)
-		(stroke
-			(width 0)
-			(type default)
-		)
-	)
-	(wire
-		(pts
 			(xy 50.8 74.93) (xy 67.31 74.93)
 		)
@@
 	(wire
 		(pts
-			(xy 224.79 69.85) (xy 224.79 68.58)
+			(xy 44.45 102.87) (xy 54.61 102.87)
 		)
 		(stroke
@@
 	(wire
 		(pts
-			(xy 44.45 102.87) (xy 54.61 102.87)
+			(xy 236.22 128.27) (xy 236.22 135.89)
 		)
 		(stroke
@@
 	(wire
 		(pts
+			(xy 245.11 125.73) (xy 245.11 143.51)
+		)
+		(stroke
+			(width 0)
+			(type default)
+		)
+	)
+	(wire
+		(pts
+			(xy 224.79 128.27) (xy 236.22 128.27)
+		)
+		(stroke
+			(width 0)
+			(type default)
+		)
+	)
+	(wire
+		(pts
+			(xy 246.38 125.73) (xy 245.11 125.73)
+		)
+		(stroke
+			(width 0)
+			(type default)
+		)
+	)
+	(wire
+		(pts
 			(xy 213.36 128.27) (xy 224.79 128.27)
 		)
@@
 		)
 	)
-	(wire
-		(pts
-			(xy 224.79 68.58) (xy 229.87 68.58)
-		)
+	(text_box "R1: ER\nR2:\nR3:\nR4: CS0402KRX7R7BB104\nR5: ERJXGNF1003Y\nR6: ERJXGNF4023Y\n\nC1: CC0402KRX5R7BB225 2u2  10% 16V\nC2: CS0402KRX7R7BB104 0u1  10% 16V\nC3: CC1206KKX5R7BB226 22u  10% 16V\nC4: CS0402KRX7R7BB104 0u1  10% 16V\nC5: CS1206JKNPOCBN470 47p  5%  1KV\nC6: CS0603KRX7R9BB472 4n7  10% 50V\nC7: CC1210MKX5R5BB107 100u 20% 6.3V\nC8: CC1210MKX5R7BB476 47u  20% 16V"
+		(exclude_from_sim yes)
+		(at 228.346 76.962 0)
+		(size 43.434 34.29)
 		(stroke
 			(width 0)
 			(type default)
 		)
+		(fill
+			(type none)
+		)
+		(effects
+			(font
+				(size 1.27 1.27)
+			)
+			(justify left top)
+		)
 	)
-	(text_box "R4: CS0402KRX7R7BB104\nC1: CC0402KRX5R7BB225\nC2: CS0402KRX7R7BB104\nC3: CC1206KKX5R7BB226\nC4: C2\nC5: C0805F473K1RACTU\nC6: CS0603KRX7R9BB472"
+	(text_box "C7+C8 = 150u\n\nR5 = 100k\nR6 = 400k\nV_REF = 0.8 V\n\nV_OUT = V_REF * (1+(R5/R6)) = 1 V\nI_OUT = V_OUT / (R5 + R6) = 2 uA\n\nP_R5 = (I_OUT)²  * R5 = 0.4 uW\nP_R5 = (I_OUT)²  * R6 = 1.6 uW"
 		(exclude_from_sim no)
-		(at 65.786 27.178 0)
-		(size 29.21 20.574)
+		(at 92.456 45.466 0)
+		(size 40.132 25.654)
 		(stroke
 			(width 0)
@@
 	(symbol
 		(lib_id "power:GND")
-		(at 224.79 69.85 0)
+		(at 245.11 143.51 0)
 		(unit 1)
 		(exclude_from_sim no)
@@
 		(fields_autoplaced yes)
 		(property "Reference" "#PWR09"
-			(at 224.79 76.2 0)
+			(at 245.11 149.86 0)
 			(effects
 				(font
@@
 		)
 		(property "Value" "GND"
-			(at 224.79 74.93 0)
+			(at 245.11 148.59 0)
 			(effects
 				(font
@@
 		)
 		(property "Footprint" ""
-			(at 224.79 69.85 0)
+			(at 245.11 143.51 0)
 			(effects
 				(font
@@
 		)
 		(property "Datasheet" ""
-			(at 224.79 69.85 0)
+			(at 245.11 143.51 0)
 			(effects
 				(font
@@
 		)
 		(property "Description" "Power symbol creates a global label with name \"GND\" , ground"
-			(at 224.79 69.85 0)
+			(at 245.11 143.51 0)
 			(effects
 				(font
@@
 	)
 	(symbol
+		(lib_id "power:GND")
+		(at 236.22 143.51 0)
+		(unit 1)
+		(exclude_from_sim no)
+		(in_bom yes)
+		(on_board yes)
+		(dnp no)
+		(fields_autoplaced yes)
+		(property "Reference" "#PWR012"
+			(at 236.22 149.86 0)
+			(effects
+				(font
+					(size 1.27 1.27)
+				)
+				(hide yes)
+			)
+		)
+		(property "Value" "GND"
+			(at 236.22 148.59 0)
+			(effects
+				(font
+					(size 1.27 1.27)
+				)
+			)
+		)
+		(property "Footprint" ""
+			(at 236.22 143.51 0)
+			(effects
+				(font
+					(size 1.27 1.27)
+				)
+				(hide yes)
+			)
+		)
+		(property "Datasheet" ""
+			(at 236.22 143.51 0)
+			(effects
+				(font
+					(size 1.27 1.27)
+				)
+				(hide yes)
+			)
+		)
+		(property "Description" "Power symbol creates a global label with name \"GND\" , ground"
+			(at 236.22 143.51 0)
+			(effects
+				(font
+					(size 1.27 1.27)
+				)
+				(hide yes)
+			)
+		)
+		(pin "1"
+		)
+		(instances
+			(project ""
+				(path "/d672ea38-1e2e-4086-a213-35bc1969a11a"
+					(reference "#PWR012")
+					(unit 1)
+				)
+			)
+		)
+	)
+	(symbol
 		(lib_id "Device:C")
 		(at 67.31 78.74 0)
@@
 			)
 		)
-		(property "Value" "150u"
+		(property "Value" "100u"
 			(at 228.6 140.9699 0)
 			(effects
@@
 			)
 		)
-		(property "Footprint" ""
+		(property "Footprint" "Capacitor_SMD:C_1210_3225Metric"
 			(at 225.7552 143.51 0)
 			(effects
@@
 	(symbol
 		(lib_id "Connector:Screw_Terminal_01x02")
-		(at 234.95 74.93 0)
+		(at 251.46 125.73 0)
 		(unit 1)
 		(exclude_from_sim no)
@@
 		(fields_autoplaced yes)
 		(property "Reference" "J1"
-			(at 237.49 74.9299 0)
+			(at 254 125.7299 0)
 			(effects
 				(font
@@
 		)
 		(property "Value" "1725656"
-			(at 237.49 77.4699 0)
+			(at 254 128.2699 0)
 			(effects
 				(font
@@
 		)
 		(property "Footprint" "TerminalBlock_Phoenix:TerminalBlock_Phoenix_MKDS-1,5-2-5.08_1x02_P5.08mm_Horizontal"
-			(at 234.95 74.93 0)
+			(at 251.46 125.73 0)
 			(effects
 				(font
@@
 		)
 		(property "Datasheet" "~"
-			(at 234.95 74.93 0)
+			(at 251.46 125.73 0)
 			(effects
 				(font
@@
 		)
 		(property "Description" "Generic screw terminal, single row, 01x02, script generated (kicad-library-utils/schlib/autogen/connector/)"
-			(at 234.95 74.93 0)
+			(at 251.46 125.73 0)
 			(effects
 				(font
@@
 					(unit 1)
 				)
+			)
+		)
+	)
+	(symbol
+		(lib_id "Device:C")
+		(at 236.22 139.7 0)
+		(unit 1)
+		(exclude_from_sim no)
+		(in_bom yes)
+		(on_board yes)
+		(dnp no)
+		(fields_autoplaced yes)
+		(property "Reference" "C8"
+			(at 240.03 138.4299 0)
+			(effects
+				(font
+					(size 1.27 1.27)
+				)
+				(justify left)
+			)
+		)
+		(property "Value" "47u"
+			(at 240.03 140.9699 0)
+			(effects
+				(font
+					(size 1.27 1.27)
+				)
+				(justify left)
+			)
+		)
+		(property "Footprint" "Capacitor_SMD:C_1210_3225Metric"
+			(at 237.1852 143.51 0)
+			(effects
+				(font
+					(size 1.27 1.27)
+				)
+				(hide yes)
+			)
+		)
+		(property "Datasheet" "~"
+			(at 236.22 139.7 0)
+			(effects
+				(font
+					(size 1.27 1.27)
+				)
+				(hide yes)
+			)
+		)
+		(property "Description" "Unpolarized capacitor"
+			(at 236.22 139.7 0)
+			(effects
+				(font
+					(size 1.27 1.27)
+				)
+				(hide yes)
+			)
+		)
+		(pin "2"
+		)
+		(pin "1"
+		)
+		(instances
+			(project ""
+				(path "/d672ea38-1e2e-4086-a213-35bc1969a11a"
+					(reference "C8")
+					(unit 1)
+				)
