File: step-down/step-down.kicad_sch (KiCad schematic)
At the start: 21 parts, among them J0 1725656, J1 1725656, M1 IRF7413ZPBF, M2 IRF7413ZPBF, U1 LTC3807EFE-TRPBF

Commit message: formattin
Parts:
- C1: value 2.2u -> 2u2
- C2, C4: value 0.1u -> 0u1
- C6: value 4.7n -> 4n7
- R2: value 15.4k -> 15k4
- R3: value 60.4k -> 60k4
Changed lines of the file:
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@@
 		)
 	)
-	(text_box "R1: ERJ-XGNF1003Y        1% 31mW\nR2: ERJ-XGNF1542Y        1% 31mW\nR3: ERJ-XGNF6042Y        1% 31mW\nR4: KRL6432D-C-R004-F-T5 1% 3.0W\nR5: ERJ-XGNF1003Y        1% 31mW\nR6: ERJ-XGNF4023Y        1% 31mW\n\nC1: CC0402KRX5R7BB225 2u2  10% 16V\nC2: CS0402KRX7R7BB104 0u1  10% 16V\nC3: CC1206KKX5R7BB226 22u  10% 16V\nC4: CS0402KRX7R7BB104 0u1  10% 16V\nC5: CS1206JKNPOCBN470 47p  5%  1KV\nC6: CS0603KRX7R9BB472 4n7  10% 50V\nC7: CC1210MKX5R5BB107 100u 20% 6.3V\nC8: CC1210MKX5R7BB476 47u  20% 16V"
+	(text_box "R1: ERJ-XGNF1003Y           1% 31mW\nR2: ERJ-XGNF1542Y           1% 31mW\nR3: ERJ-XGNF6042Y           1% 31mW\nR4: KRL6432D-C-R004-F-T5    1% 3.0W\nR5: ERJ-XGNF1003Y           1% 31mW\nR6: ERJ-XGNF4023Y           1% 31mW\n\nC1: CC0402KRX5R7BB225 2u2   10% 16V\nC2: CS0402KRX7R7BB104 0u1   10% 16V\nC3: CC1206KKX5R7BB226 22u   10% 16V\nC4: CS0402KRX7R7BB104 0u1   10% 16V\nC5: CS1206JKNPOCBN470 47p   5%  1KV\nC6: CS0603KRX7R9BB472 4n7   10% 50V\nC7: CC1210MKX5R5BB107 100u  20% 6.3V\nC8: CC1210MKX5R7BB476 47u   20% 16V"
 		(exclude_from_sim yes)
 		(at 146.05 36.83 0)
-		(size 50.546 32.004)
+		(size 55.626 34.29)
 		(stroke
 			(width 0)
@@
 			)
 		)
-		(property "Value" "0.1u"
+		(property "Value" "0u1"
 			(at 180.34 80.01 90)
 			(effects
@@
 			)
 		)
-		(property "Value" "0.1u"
+		(property "Value" "0u1"
 			(at 58.42 86.36 90)
 			(effects
@@
 			)
 		)
-		(property "Value" "2.2u"
+		(property "Value" "2u2"
 			(at 144.78 81.28 0)
 			(effects
@@
 			)
 		)
-		(property "Value" "60.4k"
+		(property "Value" "60k4"
 			(at 58.42 99.06 90)
 			(effects
@@
 			)
 		)
-		(property "Value" "15.4k"
+		(property "Value" "15k4"
 			(at 62.23 119.38 90)
 			(effects
@@
 			)
 		)
-		(property "Value" "4.7n"
+		(property "Value" "4n7"
 			(at 54.61 118.11 90)
 			(effects
