File: step-down/step-down.kicad_sch (KiCad schematic)
At the start: 21 parts, among them J0 1725656, J1 1725656, M1 IRF7413ZPBF, M2 IRF7413ZPBF, U1 LTC3807EFE-TRPBF

Commit message: assigned footprints
Parts:
- removed U1: LTC3807EFE-TRPBF, TSSOP-20_FE/CB_LIT, symbol 2025-02-07_09-07-09:LTC3807EFE-TRPBF
- added U1: LTC3807EFE-TRPBF, TSSOP-20_FE/CB_LIT, symbol LTC3807EFE-TRPBF:LTC3807EFE-TRPBF
- M1, M2: footprint SOIC127P600X175-8N -> footprint-libraries:SOIC127P600X175-8N
- R1, R5: footprint (none) -> footprint-libraries:RES_ERJXGNF1003Y
- R2: footprint (none) -> footprint-libraries:RES_ERJXGNF1542Y
- R3: footprint (none) -> footprint-libraries:RES_ERJXGNF6042Y
- R4: footprint (none) -> footprint-libraries:RESC310X630X70N
- R6: footprint (none) -> footprint-libraries:RES_ERJXGNF4023Y
Connections:
- net GND: now also U1.17 (EXTVCC)
- net GNDPWR: now also U1.18 (PGND)
- net GNDS: now also U1.4 (SGND), U1.5 (SGND)
- net at C4.2: now also U1.1 (TRACK/SS)
- net at C5.2, R2.2: now also U1.10 (ITH)
- net at R1.1: now also U1.11 (PGOOD)
- net at M1.4 (G): now also U1.12 (TG)
- net at C2.1, L1.1, M1.3 (S_3)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: now also U1.13 (SW)
- net at C2.2, D1.1: now also U1.14 (BOOST)
- net at M2.4 (G): now also U1.15 (BG)
- net at C1.2, D1.2: now also U1.16 (INTVCC)
- net at C3.1, J0.2 (Pin_2), M1.5 (D_1): now also U1.19 (VIN)
- net at R3.2: now also U1.2 (FREQ)
- net at C7.1, C8.1, J1.2 (Pin_2)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: now also U1.7 (SENSE-)
- net at L1.2, R4.1: now also U1.8 (SENSE+)
- net at R5.2, R6.1: now also U1.9 (VFB)
Changed lines of the file:
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@@
 	)
 	(junction
-		(at 71.12 123.19)
+		(at 44.45 102.87)
 		(diameter 0)
 		(color 0 0 0 0)
 	)
 	(junction
-		(at 44.45 102.87)
+		(at 71.12 123.19)
 		(diameter 0)
 		(color 0 0 0 0)
@@
 	)
 	(symbol
-		(lib_id "2025-02-07_09-07-09:LTC3807EFE-TRPBF")
-		(at 71.12 100.33 0)
-		(unit 1)
-		(exclude_from_sim no)
-		(in_bom yes)
-		(on_board yes)
-		(dnp no)
-		(fields_autoplaced yes)
-		(property "Reference" "U1"
-			(at 109.22 90.17 0)
-			(effects
-				(font
-					(size 1.524 1.524)
-				)
-			)
-		)
-		(property "Value" "LTC3807EFE-TRPBF"
-			(at 109.22 92.71 0)
-			(effects
-				(font
-					(size 1.524 1.524)
-				)
-			)
-		)
-		(property "Footprint" "TSSOP-20_FE/CB_LIT"
-			(at 71.12 100.33 0)
-			(effects
-				(font
-					(size 1.27 1.27)
-					(italic yes)
-				)
-				(hide yes)
-			)
-		)
-		(property "Datasheet" "LTC3807EFE-TRPBF"
-			(at 71.12 100.33 0)
-			(effects
-				(font
-					(size 1.27 1.27)
-					(italic yes)
-				)
-				(hide yes)
-			)
-		)
-		(property "Description" ""
-			(at 71.12 100.33 0)
-			(effects
-				(font
-					(size 1.27 1.27)
-				)
-				(hide yes)
-			)
-		)
-		(pin "8"
-		)
-		(pin "16"
-		)
-		(pin "6"
-		)
-		(pin "3"
-		)
-		(pin "7"
-		)
-		(pin "5"
-		)
-		(pin "4"
-		)
-		(pin "20"
-		)
-		(pin "1"
-		)
-		(pin "9"
-		)
-		(pin "EPAD"
-		)
-		(pin "17"
-		)
-		(pin "2"
-		)
-		(pin "18"
-		)
-		(pin "15"
-		)
-		(pin "14"
-		)
-		(pin "10"
-		)
-		(pin "11"
-		)
-		(pin "12"
-		)
-		(pin "13"
-		)
-		(pin "19"
-		)
-		(instances
-			(project ""
-				(path "/d672ea38-1e2e-4086-a213-35bc1969a11a"
-					(reference "U1")
-					(unit 1)
-				)
-			)
-		)
-	)
-	(symbol
 		(lib_id "Device:C")
 		(at 180.34 85.09 270)
@@
 			)
 		)
-		(property "Footprint" "SOIC127P600X175-8N"
+		(property "Footprint" "footprint-libraries:SOIC127P600X175-8N"
 			(at 214.63 174.93 0)
 			(effects
@@
 			)
 		)
-		(property "Footprint" ""
+		(property "Footprint" "footprint-libraries:RES_ERJXGNF4023Y"
 			(at 211.582 139.7 90)
 			(effects
@@
 			)
 		)
-		(property "Footprint" ""
+		(property "Footprint" "footprint-libraries:RESC310X630X70N"
 			(at 204.47 130.048 90)
 			(effects
@@
 			)
 		)
-		(property "Footprint" ""
+		(property "Footprint" "footprint-libraries:RES_ERJXGNF6042Y"
 			(at 58.42 104.648 90)
 			(effects
@@
 			)
 		)
-		(property "Footprint" ""
+		(property "Footprint" "footprint-libraries:RES_ERJXGNF1003Y"
 			(at 211.582 132.08 90)
 			(effects
@@
 			)
 		)
-		(property "Footprint" "SOIC127P600X175-8N"
+		(property "Footprint" "footprint-libraries:SOIC127P600X175-8N"
 			(at 214.63 202.87 0)
 			(effects
@@
 			)
 		)
-		(property "Footprint" ""
+		(property "Footprint" "footprint-libraries:RES_ERJXGNF1542Y"
 			(at 62.23 124.968 90)
 			(effects
@@
 			)
 		)
-		(property "Footprint" ""
+		(property "Footprint" "footprint-libraries:RES_ERJXGNF1003Y"
 			(at 152.4 127.508 90)
 			(effects
@@
 					(unit 1)
 				)
+			)
+		)
+	)
+	(symbol
+		(lib_id "LTC3807EFE-TRPBF:LTC3807EFE-TRPBF")
+		(at 71.12 100.33 0)
+		(unit 1)
+		(exclude_from_sim no)
+		(in_bom yes)
+		(on_board yes)
+		(dnp no)
+		(fields_autoplaced yes)
+		(property "Reference" "U1"
+			(at 109.22 90.17 0)
+			(effects
+				(font
+					(size 1.524 1.524)
+				)
+			)
+		)
+		(property "Value" "LTC3807EFE-TRPBF"
+			(at 109.22 92.71 0)
+			(effects
+				(font
+					(size 1.524 1.524)
+				)
+			)
+		)
+		(property "Footprint" "TSSOP-20_FE/CB_LIT"
+			(at 71.12 100.33 0)
+			(effects
+				(font
+					(size 1.27 1.27)
+					(italic yes)
+				)
+				(hide yes)
+			)
+		)
+		(property "Datasheet" "LTC3807EFE-TRPBF"
+			(at 71.12 100.33 0)
+			(effects
+				(font
+					(size 1.27 1.27)
+					(italic yes)
+				)
+				(hide yes)
+			)
+		)
+		(property "Description" ""
+			(at 71.12 100.33 0)
+			(effects
+				(font
+					(size 1.27 1.27)
+				)
+				(hide yes)
+			)
+		)
+		(pin "16"
+		)
+		(pin "19"
+		)
+		(pin "5"
+		)
+		(pin "6"
+		)
+		(pin "2"
+		)
+		(pin "9"
+		)
+		(pin "12"
+		)
+		(pin "18"
+		)
+		(pin "14"
+		)
+		(pin "8"
+		)
+		(pin "7"
+		)
+		(pin "10"
+		)
+		(pin "EPAD"
+		)
+		(pin "17"
+		)
+		(pin "4"
+		)
+		(pin "11"
+		)
+		(pin "13"
+		)
+		(pin "15"
+		)
+		(pin "20"
+		)
+		(pin "1"
+		)
+		(pin "3"
+		)
+		(instances
+			(project ""
+				(path "/d672ea38-1e2e-4086-a213-35bc1969a11a"
+					(reference "U1")
+					(unit 1)
+				)

Commit message: assigned footprint L1: Bourns SRP6060FA
Parts:
- L1: footprint (none) -> Inductor_SMD:L_Bourns_SRP6060FA
Changed lines of the file:
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@@
 			)
 		)
-		(property "Footprint" ""
+		(property "Footprint" "Inductor_SMD:L_Bourns_SRP6060FA"
 			(at 193.04 128.27 0)
 			(effects
