File: step-down/step-down/step-down.kicad_pcb (KiCad board)
At the start: 2 copper layers, 20 parts, among them IC1 LTC3807EFE#PBF, IC2 IRF7413ZPBF, IC3 IRF7413ZPBF, J1 Screw_Terminal_01x02, J2 Screw_Terminal_01x02

Commit message: small change
Parts:
- moved L1 20.1 mm to (155.9, 102.5)
- moved Cout1 10.6 mm to (143.9, 88.0)
- moved IC1 5.70 mm to (138.1, 98.5)
Changed lines of the file:
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@@
 	(footprint "footprints:AISC-1008F-100G-T"
 		(layer "F.Cu")
-		(at 141.9943 88.0091)
+		(at 155.855 102.5)
 		(descr "AISC-1008F-100G-T-2")
 		(tags "Inductor")
@@
 	(footprint "footprints:TAZH157J010LBSZ0H00"
 		(layer "F.Cu")
-		(at 138.7743 97.2291)
+		(at 143.9 88)
 		(descr "case size H")
 		(tags "Capacitor Polarised")
@@
 	(footprint "footprints:LTC3807EFE#PBF"
 		(layer "F.Cu")
-		(at 138.1243 104.1991)
+		(at 138.1243 98.5)
 		(descr "20-Lead Plastic TSSOP (4.4mm)")
 		(tags "Integrated Circuit")
