File: step-down2/step-down.kicad_pcb (KiCad board)
At the start: 2 copper layers, 20 parts, among them IC1 LTC3807EFE#PBF, IC2 IRF7413ZPBF, IC3 IRF7413ZPBF, J1 Screw_Terminal_01x02, J2 Screw_Terminal_01x02

Commit message: fixed all ERC errors
Parts:
- added D2: CMDSH2-3, footprints:CMDSH2-3_TR_PBFREE, F.Cu at (119.8, 70.0)
- renumbered C4 to C5, C5 to C6, IC2 to M1, IC3 to M2
Connections:
- C6 pad 2: Net-(IC1-SW) -> Net-(D2-K)
- Cout1 pad 2: unconnected-(Cout1-Pad2) -> GND
- IC1 pad 13: Net-(IC1-SW) -> Net-(D2-K)
- IC1 pad 18: GNDPWR -> GND
- L1 pad 1: Net-(IC1-SW) -> Net-(D2-K)
- M1 pad 1: Net-(IC1-SW) -> Net-(D2-K)
- M1 pad 2: unconnected-(IC2-S_2-Pad2) -> Net-(D2-K)
- M1 pad 3: unconnected-(IC2-S_3-Pad3) -> Net-(D2-K)
- M1 pad 6: unconnected-(IC2-D_2-Pad6) -> Net-(M1-D_2)
- M1 pad 7: unconnected-(IC2-D_3-Pad7) -> Net-(M1-D_2)
- M1 pad 8: unconnected-(IC2-D_4-Pad8) -> Net-(M1-D_2)
- M2 pad 1: unconnected-(IC3-S_1-Pad1) -> GND
- M2 pad 2: unconnected-(IC3-S_2-Pad2) -> GND
- M2 pad 3: unconnected-(IC3-S_3-Pad3) -> GND
- M2 pad 5: Net-(IC1-SW) -> Net-(D2-K)
- M2 pad 6: unconnected-(IC3-D_2-Pad6) -> Net-(M2-D_2)
- M2 pad 7: unconnected-(IC3-D_3-Pad7) -> Net-(M2-D_2)
- M2 pad 8: unconnected-(IC3-D_4-Pad8) -> Net-(M2-D_2)
