File: step-down-new/step-down.kicad_sch (KiCad schematic)
At the start: 22 parts, among them IC1 LTC3807EFE#PBF, J1 Screw_Terminal_01x02, J2 Screw_Terminal_01x02, M1 IRF7413ZPBF, M2 IRF7413ZPBF

Commit message: new version
Parts:
- C4: footprint C0402 -> Capacitor_SMD:C_0402_1005Metric
- R1: footprint footprints:ERJ-XGNF1542Y -> Resistor_SMD:R_01005_0402Metric
- R2: footprint footprints:ERJ-XGNF6042Y -> Resistor_SMD:R_01005_0402Metric
- R3, R5: footprint footprints:ERJ-XGNF1003Y -> Resistor_SMD:R_01005_0402Metric
- R6: footprint footprints:ERJ-XGNF4023Y -> Resistor_SMD:R_01005_0402Metric
Connections:
- net GNDPWR is gone; now on net GND: J1.1 (Pin_1)
- net GNDS is gone; now on net GND: IC1.21 (SGND_3), IC1.4 (SGND_1), IC1.5 (SGND_2)
- net SW: now reaches C5.2, D2.1 (K), IC1.13 (SW), L1.1, M1.1 (S_1), M1.2 (S_2), M1.3 (S_3), M2.5 (D_1), M2.6 (D_2), M2.7 (D_3), M2.8 (D_4)
- net SENSE+: now reaches C4.1, IC1.8 (SENSE+), L1.2, R4.1
- net SENSE-: now reaches C4.2, Cout1.1, IC1.7 (SENSE-), J2.2 (Pin_2), R4.2, R5.1
- net VFB: now reaches IC1.9 (VFB), R5.2, R6.1
- net VIN: now reaches Cin1.1, IC1.19 (VIN), J1.2 (Pin_2), M1.5 (D_1), M1.6 (D_2), M1.7 (D_3), M1.8 (D_4)
- net INTVCC: now reaches C_INTVCC1.1, D1.2 (A), IC1.16 (INTVCC), R3.1
- net PGOOD: now reaches IC1.11 (PGOOD), R3.2
- net BG: now reaches IC1.15 (BG), M2.4 (G)
- net BOOST: now reaches C5.1, D1.1 (K), IC1.14 (BOOST)
- net TG: now reaches IC1.12 (TG), M1.4 (G)
- net TRACK/SS: now reaches C2.2, IC1.1 (TRACK/SS)
- net ITH: now reaches C3.1, IC1.10 (ITH), R1.2
- net FREQ: now reaches IC1.2 (FREQ), R2.2
Other:
- moved on the sheet: R3
